File: Drone_PCB_FC/Blackbox-flash.kicad_sch (KiCad schematic)
At the start: 5 parts, among them U7 W25Q128JVE

Commit message: starting the PCB layout
Parts:
- C23: footprint (none) -> Capacitor_SMD:C_0805_2012Metric
- R10, R11, R12: footprint (none) -> Resistor_SMD:R_0805_2012Metric
Changed lines of the file:
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@@
 			)
 		)
-		(property "Footprint" ""
+		(property "Footprint" "Resistor_SMD:R_0805_2012Metric"
 			(at 102.87 100.838 90)
 			(hide yes)
@@
 			)
 		)
-		(property "Footprint" ""
+		(property "Footprint" "Resistor_SMD:R_0805_2012Metric"
 			(at 102.87 108.458 90)
 			(hide yes)
@@
 			)
 		)
-		(property "Footprint" ""
+		(property "Footprint" "Resistor_SMD:R_0805_2012Metric"
 			(at 115.062 77.47 90)
 			(hide yes)
@@
 			)
 		)
-		(property "Footprint" ""
+		(property "Footprint" "Capacitor_SMD:C_0805_2012Metric"
 			(at 141.9352 80.01 0)
 			(hide yes)
