File: Drone_PCB_FC/Blackbox-flash.kicad_sch (KiCad schematic)
At the start: 5 parts, among them U3 W25Q128JVSIQTR

Commit message: Ordered the PCB now i have to wait and see if i waisted 130 dollars
Parts:
- U3: value W25Q128JVSIQTR -> GD25Q16ETIGR; LCSC Part C97521 -> C2904431
Changed lines of the file:
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@@
 			)
 		)
-		(property "Value" "W25Q128JVSIQTR"
+		(property "Value" "GD25Q16ETIGR"
 			(at 133.35 87.63 0)
 			(show_name no)
@@
 			)
 		)
-		(property "Datasheet" "https://lcsc.com/product-detail/FLASH_W25Q128JVSIQTR_C97521.html"
+		(property "Datasheet" "https://lcsc.com/product-https://www.lcsc.com/datasheet/C2904431.pdf?spm=wm.sxq.inf.ggs___wm.fly.bg.4.xh&lcsc_vid=E1cLVgVQFFBaAgBWEgdcBV1QEVdXVVQATwAIUAJRQ1gxVlNeQ1VaV11TRVJaUTsOAxUeFF5JWBYZEEoKFBINSQcJGk4eFQsCAgIaSgADAwAHC0slRlZXVlNXWQkaCgg%3D"
 			(at 133.35 110.49 0)
 			(hide yes)
@@
 			)
 		)
-		(property "LCSC Part" "C97521"
+		(property "LCSC Part" "C2904431"
 			(at 133.35 118.11 0)
 			(hide yes)
