File: Drone_PCB_FC/Drone_PCB_FC.kicad_pcb (KiCad board)
At the start: 4 copper layers, 80 x 80 mm, 83 parts, among them CN1 SM10B-SRSS-TB, J1 Conn_01x05, J2 USB_C_Receptacle_USB2.0_14P, J3 Conn_01x04, J4 Conn_01x04, J5 Conn_01x04, J6 Conn_01x04, J7 Conn_01x06, Q2 2N7000, SW1 SW_Push, SW2 SW_Push, U1 AP2112K-3.3, U2 USBLC6-2SC6, U3 GD25Q16ETIGR, U4 STM32F405RGTx, U5 TPS5430DDAR, U7 BMI270, Y1 8MHz

Commit message: I have the test bench working. now i need the frame
Other:
- board text removed: "3.24k"
Changed lines of the file:
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@@
 		)
 	)
-	(gr_text "3.24k"
+	(gr_text "10k\n"
 		(at 174.25 120 90)
 		(layer "F.SilkS")
